Commit message: Added unthreaded cap from CAD file, modified dynamics to incorporate concave geometry (collision triangles)

File: examples/05-kuka_screwing/kuka_iiwa.urdf (robot description, URDF)
Before this commit: robot kuka_iiwa, 8 links, 7 joints
Links:
- link link6: geometry collision mesh filename=Cap_NoThreads.obj scale=0.07 0.07 0.07; visual box size=0.02 0.3 0.03

Commit message: Added constant downwards and sideways forces to maintain contact with bottle. Increased cap scale slightly so it fits over bottle lip.

File: examples/05-kuka_screwing/kuka_iiwa.urdf (robot description, URDF)
Before this commit: robot kuka_iiwa, 8 links, 7 joints
Links:
- link link6: geometry collision mesh filename=Cap_NoThreads.obj scale=0.041 0.041 0.041; visual box size=0.02 0.15 0.005
