Commit message: Modified URDF files to show bottle and cap shapes

File: examples/05-kuka_screwing/bottle.urdf (robot description, URDF)
Before this commit: robot bottle, 3 links, 2 joints
Links:
- link link1: geometry collision cylinder length=0.4 radius=0.125; visual cylinder length=0.4 radius=0.125
Joints:
- joint j0: limit lower=-2.967 upper=2.967 effort=176 velocity=1.7104 -> lower=-2.967 upper=2.967 effort=176 velocity=0
- joint j1: limit lower=-2.0944 upper=2.0944 effort=176 velocity=1.7104 -> lower=-2.0944 upper=2.0944 effort=176 velocity=0

File: examples/05-kuka_screwing/kuka_iiwa.urdf (robot description, URDF)
Before this commit: robot kuka_iiwa, 8 links, 7 joints
Links:
- link link6: geometry collision cylinder length=0.05 radius=0.125; visual cylinder length=0.05 radius=0.125

Commit message: Modified cap and bottle shapes, added code from motion control primitive to be incorporated

File: examples/05-kuka_screwing/bottle.urdf (robot description, URDF)
Before this commit: robot bottle, 3 links, 2 joints
Links:
- link link1: geometry collision cylinder length=0.2 radius=0.06; visual cylinder length=0.2 radius=0.06

Commit message: Limited screwing to begin based on a force threshold and end after a threshold angle has been reached

File: examples/05-kuka_screwing/bottle.urdf (robot description, URDF)
Before this commit: robot bottle, 3 links, 2 joints
Links:
- link link1: geometry collision cylinder length=0.25 radius=0.06; visual cylinder length=0.25 radius=0.06

Commit message: Added bottle CAD, created a motion primitive approach method

File: examples/05-kuka_screwing/bottle.urdf (robot description, URDF)
Before this commit: robot bottle, 3 links, 2 joints
Links:
- link link1: geometry collision mesh filename=Bottle_NoThreads.obj scale=0.04 0.04 0.04; visual mesh filename=Bottle_NoThreads.obj scale=0.04 0.04 0.04

File: examples/05-kuka_screwing/kuka_iiwa.urdf (robot description, URDF)
Before this commit: robot kuka_iiwa, 8 links, 7 joints
Links:
- link link6: geometry collision mesh filename=Cap_NoThreads.obj scale=0.04 0.04 0.04; visual box size=0.02 0.15 0.01

Commit message: Modified alignment strategy, fixed screwing, tuned gains

File: examples/05-kuka_screwing/bottle.urdf (robot description, URDF)
Before this commit: robot bottle, 3 links, 2 joints
Links:
- link link1: geometry collision cylinder length=0.22 radius=0.045; visual cylinder length=0.21 radius=0.055

File: examples/05-kuka_screwing/kuka_iiwa.urdf (robot description, URDF)
Before this commit: robot kuka_iiwa, 8 links, 7 joints
Links:
- link link6: geometry collision mesh filename=Cap2_NoThreads.obj scale=0.041 0.041 0.041; visual box size=0.02 0.15 0.005
