Commit message: Redoing stuff from missing commits that disappeared in branch merge. Fixed panda screwing urdf files. The controller from kuka works for panda without changing it.

File: examples/05-panda_screwing/bottle.urdf (robot description, URDF)
Before this commit: robot bottle, 3 links, 2 joints
Links:
- link link1: geometry collision cylinder length=0.22 radius=0.055; visual cylinder length=0.21 radius=0.055
