Commit message: changed the control link to 7 because panda has one more than kuka

File: examples/05-panda_screwing/panda_arm.urdf (robot description, URDF)
Before this commit: robot panda, 8 links, 7 joints
Links:
- link link7: geometry collision mesh filename=Cap2_NoThreads.obj scale=0.041 0.041 0.041; visual box size=0.02 0.15 0.005

Commit message: Made changes to gitignore file to ignore .obj and .dae object files. Fixed build errors having to do with sleep() method compatibility between mac and ubuntu (still needs to be tested on ubuntu) and Sai2Model constructor

File: examples/05-panda_screwing/panda_arm.urdf (robot description, URDF)
Before this commit: robot panda, 8 links, 7 joints
Links:
- link link0: geometry visual mesh filename=../../../../examples/models/panda/meshes/visual/link0.obj
- link link1: geometry visual mesh filename=../../../../examples/models/panda/meshes/visual/link1.obj
- link link2: geometry visual mesh filename=../../../../examples/models/panda/meshes/visual/link2.obj
- link link3: geometry visual mesh filename=../../../../examples/models/panda/meshes/visual/link3.obj
- link link4: geometry visual mesh filename=../../../../examples/models/panda/meshes/visual/link4.obj
- link link5: geometry visual mesh filename=../../../../examples/models/panda/meshes/visual/link5.obj
- link link6: geometry visual mesh filename=../../../../examples/models/panda/meshes/visual/link6.obj
- link link7: geometry collision mesh filename=Cap2_NoThreads.obj scale=0.041 0.041 0.041; visual box size=0.02 0.15 0.005
